File: KiCAD_Project/power.kicad_sch (KiCad schematic)
At the start: 16 parts, among them J11 NP_Conn_01x02_Relief, J12 NP_Conn_01x02_Relief, Q4 1-0000505, U6 1-0001649, U7 1-0000658

Commit message: Finished Revised 2.2 Layout
Parts:
- renumbered J11 to J10, J12 to J11, R36 to R37, R37 to R38
