File: KiCAD_Project/power.kicad_sch (KiCad schematic)
At the start: 16 parts, among them J10 NP_Conn_01x02_Relief, J11 NP_Conn_01x02_Relief, Q4 1-0000505, U6 1-0001649, U7 1-0000658

Commit message: Make Rev 2.3 production files
Parts:
- renumbered J11 to J10, J10 to J9, R37 to R29, R38 to R30
Changed lines of the file:
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@@
 		(on_board yes)
 		(dnp no)
-		(property "Reference" "#PWR057"
+		(property "Reference" "#PWR056"
 			(at 139.7 107.95 0)
 			(effects
@@
 			(project "Cutdown"
 				(path "/8a527631-9f08-4346-91a8-17ddc9930238/14dc79cf-03b1-4356-bd69-4f0cd3714637"
-					(reference "#PWR057")
+					(reference "#PWR056")
 					(unit 1)
 				)
@@
 		(on_board yes)
 		(dnp no)
-		(property "Reference" "#PWR054"
+		(property "Reference" "#PWR053"
 			(at 123.19 64.77 0)
 			(effects
@@
 			(project "Cutdown"
 				(path "/8a527631-9f08-4346-91a8-17ddc9930238/14dc79cf-03b1-4356-bd69-4f0cd3714637"
-					(reference "#PWR054")
+					(reference "#PWR053")
 					(unit 1)
 				)
@@
 		(on_board yes)
 		(dnp no)
-		(property "Reference" "#PWR059"
+		(property "Reference" "#PWR058"
 			(at 152.4 95.25 0)
 			(effects
@@
 			(project "Cutdown"
 				(path "/8a527631-9f08-4346-91a8-17ddc9930238/14dc79cf-03b1-4356-bd69-4f0cd3714637"
-					(reference "#PWR059")
+					(reference "#PWR058")
 					(unit 1)
 				)
@@
 		(on_board yes)
 		(dnp no)
-		(property "Reference" "#PWR061"
+		(property "Reference" "#PWR060"
 			(at 152.4 144.78 0)
 			(effects
@@
 			(project "Cutdown"
 				(path "/8a527631-9f08-4346-91a8-17ddc9930238/14dc79cf-03b1-4356-bd69-4f0cd3714637"
-					(reference "#PWR061")
+					(reference "#PWR060")
 					(unit 1)
 				)
@@
 		(on_board yes)
 		(dnp no)
-		(property "Reference" "R37"
+		(property "Reference" "R29"
 			(at 107.315 133.35 90)
 			(effects
@@
 			(project "Cutdown"
 				(path "/8a527631-9f08-4346-91a8-17ddc9930238/14dc79cf-03b1-4356-bd69-4f0cd3714637"
-					(reference "R37")
+					(reference "R29")
 					(unit 1)
 				)
@@
 		(on_board yes)
 		(dnp no)
-		(property "Reference" "#PWR053"
+		(property "Reference" "#PWR052"
 			(at 109.22 149.86 0)
 			(effects
@@
 			(project "Cutdown"
 				(path "/8a527631-9f08-4346-91a8-17ddc9930238/14dc79cf-03b1-4356-bd69-4f0cd3714637"
-					(reference "#PWR053")
+					(reference "#PWR052")
 					(unit 1)
 				)
@@
 		(on_board yes)
 		(dnp no)
-		(property "Reference" "J11"
+		(property "Reference" "J10"
 			(at 128.27 60.96 0)
 			(effects
@@
 			(project "Cutdown"
 				(path "/8a527631-9f08-4346-91a8-17ddc9930238/14dc79cf-03b1-4356-bd69-4f0cd3714637"
-					(reference "J11")
+					(reference "J10")
 					(unit 1)
 				)
@@
 		(on_board yes)
 		(dnp no)
-		(property "Reference" "#PWR065"
+		(property "Reference" "#PWR064"
 			(at 172.72 132.08 0)
 			(effects
@@
 			(project "Cutdown"
 				(path "/8a527631-9f08-4346-91a8-17ddc9930238/14dc79cf-03b1-4356-bd69-4f0cd3714637"
-					(reference "#PWR065")
+					(reference "#PWR064")
 					(unit 1)
 				)
@@
 		(on_board yes)
 		(dnp no)
-		(property "Reference" "#PWR062"
+		(property "Reference" "#PWR061"
 			(at 156.21 77.47 0)
 			(effects
@@
 			(project "Cutdown"
 				(path "/8a527631-9f08-4346-91a8-17ddc9930238/14dc79cf-03b1-4356-bd69-4f0cd3714637"
-					(reference "#PWR062")
+					(reference "#PWR061")
 					(unit 1)
 				)
@@
 		(on_board yes)
 		(dnp no)
-		(property "Reference" "#PWR056"
+		(property "Reference" "#PWR055"
 			(at 127 105.41 0)
 			(effects
@@
 			(project "Cutdown"
 				(path "/8a527631-9f08-4346-91a8-17ddc9930238/14dc79cf-03b1-4356-bd69-4f0cd3714637"
-					(reference "#PWR056")
+					(reference "#PWR055")
 					(unit 1)
 				)
@@
 		(on_board yes)
 		(dnp no)
-		(property "Reference" "#PWR064"
+		(property "Reference" "#PWR063"
 			(at 166.37 59.69 0)
 			(effects
@@
 			(project "Cutdown"
 				(path "/8a527631-9f08-4346-91a8-17ddc9930238/14dc79cf-03b1-4356-bd69-4f0cd3714637"
-					(reference "#PWR064")
+					(reference "#PWR063")
 					(unit 1)
 				)
@@
 		(on_board yes)
 		(dnp no)
-		(property "Reference" "#PWR060"
+		(property "Reference" "#PWR059"
 			(at 152.4 105.41 0)
 			(effects
@@
 			(project "Cutdown"
 				(path "/8a527631-9f08-4346-91a8-17ddc9930238/14dc79cf-03b1-4356-bd69-4f0cd3714637"
-					(reference "#PWR060")
+					(reference "#PWR059")
 					(unit 1)
 				)
@@
 		(on_board yes)
 		(dnp no)
-		(property "Reference" "R38"
+		(property "Reference" "R30"
 			(at 154.305 68.58 90)
 			(effects
@@
 			(project "Cutdown"
 				(path "/8a527631-9f08-4346-91a8-17ddc9930238/14dc79cf-03b1-4356-bd69-4f0cd3714637"
-					(reference "R38")
+					(reference "R30")
 					(unit 1)
 				)
@@
 		(on_board yes)
 		(dnp no)
-		(property "Reference" "#PWR055"
+		(property "Reference" "#PWR054"
 			(at 127 95.25 0)
 			(effects
@@
 			(project "Cutdown"
 				(path "/8a527631-9f08-4346-91a8-17ddc9930238/14dc79cf-03b1-4356-bd69-4f0cd3714637"
-					(reference "#PWR055")
+					(reference "#PWR054")
 					(unit 1)
 				)
@@
 		(on_board yes)
 		(dnp no)
-		(property "Reference" "#PWR058"
+		(property "Reference" "#PWR057"
 			(at 139.7 142.24 0)
 			(effects
@@
 			(project "Cutdown"
 				(path "/8a527631-9f08-4346-91a8-17ddc9930238/14dc79cf-03b1-4356-bd69-4f0cd3714637"
-					(reference "#PWR058")
+					(reference "#PWR057")
 					(unit 1)
 				)
@@
 		(on_board yes)
 		(dnp no)
-		(property "Reference" "#PWR052"
+		(property "Reference" "#PWR051"
 			(at 109.22 124.46 0)
 			(effects
@@
 			(project "Cutdown"
 				(path "/8a527631-9f08-4346-91a8-17ddc9930238/14dc79cf-03b1-4356-bd69-4f0cd3714637"
-					(reference "#PWR052")
+					(reference "#PWR051")
 					(unit 1)
 				)
@@
 		(on_board yes)
 		(dnp no)
-		(property "Reference" "J10"
+		(property "Reference" "J9"
 			(at 118.11 53.34 0)
 			(effects
@@
 			(project "Cutdown"
 				(path "/8a527631-9f08-4346-91a8-17ddc9930238/14dc79cf-03b1-4356-bd69-4f0cd3714637"
-					(reference "J10")
+					(reference "J9")
 					(unit 1)
 				)
@@
 		(on_board yes)
 		(dnp no)
-		(property "Reference" "#PWR051"
+		(property "Reference" "#PWR050"
 			(at 5.08 19.05 0)
 			(effects
@@
 			(project "Cutdown"
 				(path "/8a527631-9f08-4346-91a8-17ddc9930238/14dc79cf-03b1-4356-bd69-4f0cd3714637"
-					(reference "#PWR051")
+					(reference "#PWR050")
 					(unit 1)
 				)
@@
 		(on_board yes)
 		(dnp no)
-		(property "Reference" "#PWR063"
+		(property "Reference" "#PWR062"
 			(at 165.1 142.24 0)
 			(effects
@@
 			(project "Cutdown"
 				(path "/8a527631-9f08-4346-91a8-17ddc9930238/14dc79cf-03b1-4356-bd69-4f0cd3714637"
-					(reference "#PWR063")
-					(unit 1)
-				)
+					(reference "#PWR062")
+					(unit 1)
+				)
