File: KiCAD_Project/sd_card.kicad_sch (KiCad schematic)
At the start: 4 parts, among them J9 1-0000190

Commit message: Make Rev 2.3 production files
Parts:
- renumbered J9 to J8, R35 to R27, R36 to R28
Changed lines of the file:
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@@
 		(on_board yes)
 		(dnp no)
-		(property "Reference" "#PWR047"
+		(property "Reference" "#PWR046"
 			(at 107.95 59.69 0)
 			(effects
@@
 			(project "Cutdown"
 				(path "/8a527631-9f08-4346-91a8-17ddc9930238/4ccd02fd-4bb7-4112-b550-dd4665d55a03"
-					(reference "#PWR047")
+					(reference "#PWR046")
 					(unit 1)
 				)
@@
 		(dnp no)
 		(fields_autoplaced yes)
-		(property "Reference" "J9"
+		(property "Reference" "J8"
 			(at 160.02 81.2799 0)
 			(effects
@@
 			(project "Cutdown"
 				(path "/8a527631-9f08-4346-91a8-17ddc9930238/4ccd02fd-4bb7-4112-b550-dd4665d55a03"
-					(reference "J9")
+					(reference "J8")
 					(unit 1)
 				)
@@
 		(on_board yes)
 		(dnp no)
-		(property "Reference" "#PWR049"
+		(property "Reference" "#PWR048"
 			(at 114.3 59.69 0)
 			(effects
@@
 			(project "Cutdown"
 				(path "/8a527631-9f08-4346-91a8-17ddc9930238/4ccd02fd-4bb7-4112-b550-dd4665d55a03"
-					(reference "#PWR049")
+					(reference "#PWR048")
 					(unit 1)
 				)
@@
 		(on_board yes)
 		(dnp no)
-		(property "Reference" "#PWR048"
+		(property "Reference" "#PWR047"
 			(at 107.95 101.6 0)
 			(effects
@@
 			(project "Cutdown"
 				(path "/8a527631-9f08-4346-91a8-17ddc9930238/4ccd02fd-4bb7-4112-b550-dd4665d55a03"
-					(reference "#PWR048")
+					(reference "#PWR047")
 					(unit 1)
 				)
@@
 		(on_board yes)
 		(dnp no)
-		(property "Reference" "R35"
+		(property "Reference" "R27"
 			(at 110.998 59.69 90)
 			(effects
@@
 			(project "Cutdown"
 				(path "/8a527631-9f08-4346-91a8-17ddc9930238/4ccd02fd-4bb7-4112-b550-dd4665d55a03"
-					(reference "R35")
+					(reference "R27")
 					(unit 1)
 				)
@@
 		(on_board yes)
 		(dnp no)
-		(property "Reference" "#PWR046"
+		(property "Reference" "#PWR045"
 			(at 100.33 66.04 0)
 			(effects
@@
 			(project "Cutdown"
 				(path "/8a527631-9f08-4346-91a8-17ddc9930238/4ccd02fd-4bb7-4112-b550-dd4665d55a03"
-					(reference "#PWR046")
+					(reference "#PWR045")
 					(unit 1)
 				)
@@
 		(on_board yes)
 		(dnp no)
-		(property "Reference" "R36"
+		(property "Reference" "R28"
 			(at 117.602 59.69 90)
 			(effects
@@
 			(project "Cutdown"
 				(path "/8a527631-9f08-4346-91a8-17ddc9930238/4ccd02fd-4bb7-4112-b550-dd4665d55a03"
-					(reference "R36")
+					(reference "R28")
 					(unit 1)
 				)
@@
 		(on_board yes)
 		(dnp no)
-		(property "Reference" "#PWR050"
+		(property "Reference" "#PWR049"
 			(at 121.92 109.22 0)
 			(effects
@@
 			(project "Cutdown"
 				(path "/8a527631-9f08-4346-91a8-17ddc9930238/4ccd02fd-4bb7-4112-b550-dd4665d55a03"
-					(reference "#PWR050")
-					(unit 1)
-				)
+					(reference "#PWR049")
+					(unit 1)
+				)
